Commit message: New version of ROS2 workspace

File: src/diffbot_sim/urdf/obs1.urdf.xacro (robot description, xacro)
@@ -1,4 +1,6 @@
 <?xml version="1.0"?>
-<robot xmlns:xacro="http://www.ros.org/wiki/xacro" name="leader">
+<robot xmlns:xacro="http://www.ros.org/wiki/xacro" name="$(arg robot_name)">
+  <!-- Define the dynamic robot name argument (defaults to obs1) -->
+  <xacro:arg name="robot_name" default="obs1"/>
   <xacro:macro name="inertial_sphere" params="mass radius *origin">
     <inertial>
@@ -45,8 +47,5 @@
     <color rgba="1 0.3 0.1 1"/>
   </material>
-  <material name="green">
-    <color rgba="0 1 0 1"/>
-  </material>
-  <material name="black">
+    <material name="black">
     <color rgba="0 0 0 1"/>
   </material>
@@ -72,5 +71,5 @@
         <box size="${chassis_length} ${chassis_width} ${chassis_height}"/>
       </geometry>
-      <material name="green"/>
+      <material name="black"/>
     </visual>
     <collision>
@@ -80,11 +79,10 @@
       </geometry>
     </collision>
-    <xacro:inertial_box mass="1.0"
-      x="${chassis_length}" y="${chassis_width}" z="${chassis_height}">
+    <xacro:inertial_box mass="1.0" x="${chassis_length}" y="${chassis_width}" z="${chassis_height}">
       <origin xyz="0 0 0"/>
     </xacro:inertial_box>
   </link>
   <gazebo reference="chassis">
-    <material>Gazebo/Red</material>
+    <material>Gazebo/Black</material>
   </gazebo>
   <joint name="front_left_wheel_joint" type="continuous">
@@ -196,9 +194,12 @@
     <material>Gazebo/Black</material>
   </gazebo>
+  <!-- Modified Gazebo Diff Drive Plugin -->
   <gazebo>
     <plugin filename="libgazebo_ros_diff_drive.so" name="differential_drive_controller">
       <update_rate>100</update_rate>
       <ros>
-        <namespace>/leader</namespace>
+        <!-- Puts the nodes inside a clean local namespace (e.g., /obs1) -->
+        <namespace>/$(arg robot_name)</namespace>
+        <!-- Removed the remap tag so it defaults to /obsX/cmd_vel -->
       </ros>
       <num_wheel_pairs>2</num_wheel_pairs>
@@ -217,6 +218,7 @@
       <publish_wheel_tf>true</publish_wheel_tf>
       <use_stamped_vel>false</use_stamped_vel>
-      <odometry_frame>odom</odometry_frame>
-      <robot_base_frame>leader/base_link</robot_base_frame>
+      <!-- Separate TF tree frames to avoid frame collisions -->
+      <odometry_frame>$(arg robot_name)/odom</odometry_frame>
+      <robot_base_frame>$(arg robot_name)/base_link</robot_base_frame>
     </plugin>
   </gazebo>
