Commit message: Initial commit

File: src/diffbot_sim/urdf/leader.urdf.xacro (robot description, xacro)
@@ -86,5 +86,5 @@
   </link>
   <gazebo reference="chassis">
-    <material>Gazebo/Red</material>
+    <material>Gazebo/Green</material>
   </gazebo>
   <joint name="front_left_wheel_joint" type="continuous">
